File: pcb/skibidi-phone-usb-hub.kicad_sch (KiCad schematic)
At the start: 11 parts, among them U1 FE1.1s, Y1 12Mhz

Commit message: add schematic pdf + metadata
Other:
- company: (none) -> Toby Cm's Lab x Hack Club
- title: (none) -> Skibidi Phone USB Hub
Changed lines of the file:
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@@
 	(generator_version "9.0")
 	(paper "A4")
+	(title_block
+		(title "Skibidi Phone USB Hub")
+		(date "2026-03-20")
+		(rev "V1")
+		(company "Toby Cm's Lab x Hack Club")
+	)
 	(text "Crystal"
 		(exclude_from_sim no)

Commit message: add ibom and fixes issue with power negotiation
Signed-off-by: Toby Cm <toby@vsus.app>
Parts:
- removed R1: 5.1k, Resistor_SMD:R_0603_1608Metric, symbol Device:R
Connections:
- net +3V3: no longer U1.26 (OVCJ)
- net GND: no longer U1.19 (BUSJ)
- net VBUS: now also U1.17 (~{XRSTJ}), U1.19 (BUSJ), U1.26 (OVCJ)
